Commit message: ContactSensors for collisions
Correct end effector position calculation

File: robotiq/robotiq_description/urdf/robotiq_85_gripper.urdf.xacro (robot description, xacro)
@@ -61,4 +61,18 @@
       </inertial>
     </link>
+     <gazebo reference="${prefix}robotiq_85_left_knuckle_link">
+      <sensor name="${prefix}robotiq_85_left_knuckle_link_collision_sensor" type="contact">
+        <selfCollide>true</selfCollide>
+        <always_on>true</always_on>
+        <update_rate>30</update_rate>
+        <contact>
+          <collision>${prefix}robotiq_85_left_knuckle_link_collision_sensor</collision>
+        </contact>
+        <plugin name="bumper_plugin" filename="libgazebo_ros_bumper.so">
+          <bumperTopicName>${prefix}robotiq_85_left_knuckle_link_collision_sensor</bumperTopicName>
+          <frameName>world</frameName>
+        </plugin>
+      </sensor>
+    </gazebo>
     <link name="${prefix}robotiq_85_right_knuckle_link">
       <visual>
@@ -80,4 +94,18 @@
       </inertial>
     </link>
+    <gazebo reference="${prefix}robotiq_85_right_knuckle_link">
+      <sensor name="${prefix}robotiq_85_right_knuckle_link_collision_sensor" type="contact">
+        <selfCollide>true</selfCollide>
+        <always_on>true</always_on>
+        <update_rate>30</update_rate>
+        <contact>
+          <collision>${prefix}robotiq_85_right_knuckle_link_collision_sensor</collision>
+        </contact>
+        <plugin name="bumper_plugin" filename="libgazebo_ros_bumper.so">
+          <bumperTopicName>${prefix}robotiq_85_right_knuckle_link_collision_sensor</bumperTopicName>
+          <frameName>world</frameName>
+        </plugin>
+      </sensor>
+    </gazebo>
     <joint name="${prefix}robotiq_85_left_finger_joint" type="fixed">
       <parent link="${prefix}robotiq_85_left_knuckle_link"/>
@@ -163,4 +191,18 @@
       </inertial>
     </link>
+    <gazebo reference="${prefix}robotiq_85_left_inner_knuckle_link">
+      <sensor name="${prefix}robotiq_85_left_inner_knuckle_link_collision_sensor" type="contact">
+        <selfCollide>true</selfCollide>
+        <always_on>true</always_on>
+        <update_rate>30</update_rate>
+        <contact>
+          <collision>${prefix}robotiq_85_left_inner_knuckle_link_collision_sensor</collision>
+        </contact>
+        <plugin name="bumper_plugin" filename="libgazebo_ros_bumper.so">
+          <bumperTopicName>${prefix}robotiq_85_left_inner_knuckle_link_collision_sensor</bumperTopicName>
+          <frameName>world</frameName>
+        </plugin>
+      </sensor>
+    </gazebo>
     <link name="${prefix}robotiq_85_right_inner_knuckle_link">
       <visual>
@@ -182,4 +224,18 @@
       </inertial>
     </link>
+    <gazebo reference="${prefix}robotiq_85_right_inner_knuckle_link">
+      <sensor name="${prefix}robotiq_85_right_inner_knuckle_link_collision_sensor" type="contact">
+        <selfCollide>true</selfCollide>
+        <always_on>true</always_on>
+        <update_rate>30</update_rate>
+        <contact>
+          <collision>${prefix}robotiq_85_right_inner_knuckle_link_collision_sensor</collision>
+        </contact>
+        <plugin name="bumper_plugin" filename="libgazebo_ros_bumper.so">
+          <bumperTopicName>${prefix}robotiq_85_right_inner_knuckle_link_collision_sensor</bumperTopicName>
+          <frameName>world</frameName>
+        </plugin>
+      </sensor>
+    </gazebo>
     <joint name="${prefix}robotiq_85_left_finger_tip_joint" type="continuous">
       <parent link="${prefix}robotiq_85_left_inner_knuckle_link"/>
@@ -217,4 +273,18 @@
       </inertial>
     </link>
+    <gazebo reference="${prefix}robotiq_85_left_finger_tip_link">
+      <sensor name="${prefix}robotiq_85_left_finger_tip_link_collision_sensor" type="contact">
+        <selfCollide>true</selfCollide>
+        <always_on>true</always_on>
+        <update_rate>30</update_rate>
+        <contact>
+          <collision>${prefix}robotiq_85_left_finger_tip_link_collision_sensor</collision>
+        </contact>
+        <plugin name="bumper_plugin" filename="libgazebo_ros_bumper.so">
+          <bumperTopicName>${prefix}robotiq_85_left_finger_tip_link_collision_sensor</bumperTopicName>
+          <frameName>world</frameName>
+        </plugin>
+      </sensor>
+    </gazebo>
     <link name="${prefix}robotiq_85_right_finger_tip_link">
       <visual>
@@ -236,4 +306,18 @@
       </inertial>
     </link>
+    <gazebo reference="${prefix}robotiq_85_right_finger_tip_link">
+      <sensor name="${prefix}robotiq_85_right_finger_tip_link_collision_sensor" type="contact">
+        <selfCollide>true</selfCollide>
+        <always_on>true</always_on>
+        <update_rate>30</update_rate>
+        <contact>
+          <collision>${prefix}robotiq_85_right_finger_tip_link_collision_sensor</collision>
+        </contact>
+        <plugin name="bumper_plugin" filename="libgazebo_ros_bumper.so">
+          <bumperTopicName>${prefix}robotiq_85_right_finger_tip_link_collision_sensor</bumperTopicName>
+          <frameName>world</frameName>
+        </plugin>
+      </sensor>
+    </gazebo>
     <!-- Improve grasping physics -->
     <gazebo reference="${prefix}robotiq_85_left_finger_tip_link">

File: ur5/ur5_description/urdf/ur5.urdf.xacro (robot description, xacro)
@@ -117,4 +117,18 @@
       </xacro:cylinder_inertial>
     </link>
+    <gazebo reference="${prefix}shoulder_link">
+      <sensor name="${prefix}shoulder_link_collision_sensor" type="contact">
+        <selfCollide>true</selfCollide>
+        <always_on>true</always_on>
+        <update_rate>30</update_rate>
+        <contact>
+          <collision>${prefix}upper_arm_link_collision</collision>
+        </contact>
+        <plugin name="bumper_plugin" filename="libgazebo_ros_bumper.so">
+          <bumperTopicName>${prefix}shoulder_link_collision_sensor</bumperTopicName>
+          <frameName>world</frameName>
+        </plugin>
+      </sensor>
+    </gazebo>
     <joint name="${prefix}shoulder_lift_joint" type="revolute">
       <parent link="${prefix}shoulder_link" />
@@ -148,4 +162,18 @@
       </xacro:cylinder_inertial>
     </link>
+    <gazebo reference="${prefix}upper_arm_link">
+      <sensor name="${prefix}upper_arm_link_collision_sensor" type="contact">
+        <selfCollide>true</selfCollide>
+        <always_on>true</always_on>
+        <update_rate>30</update_rate>
+        <contact>
+          <collision>${prefix}upper_arm_link_collision</collision>
+        </contact>
+        <plugin name="bumper_plugin" filename="libgazebo_ros_bumper.so">
+          <bumperTopicName>${prefix}upper_arm_link_collision_sensor</bumperTopicName>
+          <frameName>world</frameName>
+        </plugin>
+      </sensor>
+    </gazebo>
     <joint name="${prefix}elbow_joint" type="revolute">
       <parent link="${prefix}upper_arm_link" />
@@ -179,4 +207,18 @@
       </xacro:cylinder_inertial>
     </link>
+    <gazebo reference="${prefix}forearm_link">
+      <sensor name="${prefix}forearm_link_collision_sensor" type="contact">
+        <selfCollide>true</selfCollide>
+        <always_on>true</always_on>
+        <update_rate>30</update_rate>
+        <contact>
+          <collision>${prefix}forearm_link_collision</collision>
+        </contact>
+        <plugin name="bumper_plugin" filename="libgazebo_ros_bumper.so">
+          <bumperTopicName>${prefix}forearm_link_collision_sensor</bumperTopicName>
+          <frameName>world</frameName>
+        </plugin>
+      </sensor>
+    </gazebo>
     <joint name="${prefix}wrist_1_joint" type="revolute">
       <parent link="${prefix}forearm_link" />
@@ -210,4 +252,18 @@
       </xacro:cylinder_inertial>
     </link>
+    <gazebo reference="${prefix}wrist_1_link">
+      <sensor name="${prefix}wrist_1_link_collision_sensor" type="contact">
+        <selfCollide>true</selfCollide>
+        <always_on>true</always_on>
+        <update_rate>30</update_rate>
+        <contact>
+          <collision>${prefix}wrist_1_link_collision_sensor</collision>
+        </contact>
+        <plugin name="bumper_plugin" filename="libgazebo_ros_bumper.so">
+          <bumperTopicName>${prefix}wrist_1_link_collision_sensor</bumperTopicName>
+          <frameName>world</frameName>
+        </plugin>
+      </sensor>
+    </gazebo>
     <joint name="${prefix}wrist_2_joint" type="revolute">
       <parent link="${prefix}wrist_1_link" />
@@ -241,4 +297,18 @@
       </xacro:cylinder_inertial>
     </link>
+    <gazebo reference="${prefix}wrist_2_link">
+      <sensor name="${prefix}wrist_2_link_collision_sensor" type="contact">
+        <selfCollide>true</selfCollide>
+        <always_on>true</always_on>
+        <update_rate>30</update_rate>
+        <contact>
+          <collision>${prefix}wrist_2_link_collision_sensor</collision>
+        </contact>
+        <plugin name="bumper_plugin" filename="libgazebo_ros_bumper.so">
+          <bumperTopicName>${prefix}wrist_2_link_collision_sensor</bumperTopicName>
+          <frameName>world</frameName>
+        </plugin>
+      </sensor>
+    </gazebo>
     <joint name="${prefix}wrist_3_joint" type="revolute">
       <parent link="${prefix}wrist_2_link" />
@@ -272,4 +342,18 @@
       </xacro:cylinder_inertial>
     </link>
+    <gazebo reference="${prefix}wrist_3_link">
+      <sensor name="${prefix}wrist_3_link_collision_sensor" type="contact">
+        <selfCollide>true</selfCollide>
+        <always_on>true</always_on>
+        <update_rate>30</update_rate>
+        <contact>
+          <collision>${prefix}wrist_3_link_collision_sensor</collision>
+        </contact>
+        <plugin name="bumper_plugin" filename="libgazebo_ros_bumper.so">
+          <bumperTopicName>${prefix}wrist_3_link_collision_sensor</bumperTopicName>
+          <frameName>world</frameName>
+        </plugin>
+      </sensor>
+    </gazebo>
     <joint name="${prefix}ee_fixed_joint" type="fixed">
       <parent link="${prefix}wrist_3_link" />
