Commit message: Empty world (only cube)

File: ur5/ur5_description/urdf/ur5.urdf.xacro (robot description, xacro)
@@ -182,5 +182,5 @@
       <axis xyz="0 1 0" />
       <xacro:unless value="${joint_limited}">
-        <limit lower="${-pi}" upper="${pi}" effort="150.0" velocity="3.15"/>
+        <limit lower="${-0.75 * pi}" upper="${0.75 * pi}" effort="150.0" velocity="3.15"/>
       </xacro:unless>
       <xacro:if value="${joint_limited}">

File: ur5/ur5_description/urdf/ur5_robotiq85_gripper.urdf.xacro (robot description, xacro)
@@ -1,5 +1,5 @@
 <?xml version="1.0"?>
 <robot name="ur5" xmlns:xacro="http://www.ros.org/wiki/xacro">
-  <xacro:include filename="$(find ur5_description)/urdf/ur5_joint_limited_robot.urdf.xacro" />
+  <xacro:include filename="$(find ur5_description)/urdf/ur5_robot.urdf.xacro" />
   <xacro:include filename="$(find robotiq_description)/urdf/robotiq_85_gripper.urdf.xacro" />
   <!-- Robotiq Coupler -->

Commit message: General env and training updates

File: ur5/ur5_description/urdf/ur5.urdf.xacro (robot description, xacro)
@@ -86,15 +86,15 @@
       </xacro:cylinder_inertial>
     </link>
-    <joint name="${prefix}shoulder_pan_joint" type="revolute">
+    <joint name="${prefix}shoulder_pan_joint" type="continuous">
       <parent link="${prefix}base_link" />
       <child link = "${prefix}shoulder_link" />
       <origin xyz="0.0 0.0 ${shoulder_height}" rpy="0.0 0.0 0.0" />
       <axis xyz="0 0 1" />
-      <xacro:unless value="${joint_limited}">
+      <!-- <xacro:unless value="${joint_limited}">
         <limit lower="${-2.0 * pi}" upper="${2.0 * pi}" effort="150.0" velocity="3.15"/>
       </xacro:unless>
       <xacro:if value="${joint_limited}">
         <limit lower="${-pi}" upper="${pi}" effort="150.0" velocity="3.15"/>
-      </xacro:if>
+      </xacro:if> -->
       <dynamics damping="0.0" friction="0.0"/>
     </joint>
@@ -131,15 +131,15 @@
       </sensor>
     </gazebo>
-    <joint name="${prefix}shoulder_lift_joint" type="revolute">
+    <joint name="${prefix}shoulder_lift_joint" type="continuous">
       <parent link="${prefix}shoulder_link" />
       <child link = "${prefix}upper_arm_link" />
       <origin xyz="0.0 ${shoulder_offset} 0.0" rpy="0.0 ${pi / 2.0} 0.0" />
       <axis xyz="0 1 0" />
-      <xacro:unless value="${joint_limited}">
+      <!-- <xacro:unless value="${joint_limited}">
         <limit lower="${-2.0 * pi}" upper="${2.0 * pi}" effort="150.0" velocity="3.15"/>
       </xacro:unless>
       <xacro:if value="${joint_limited}">
         <limit lower="${-pi}" upper="${pi}" effort="150.0" velocity="3.15"/>
-      </xacro:if>
+      </xacro:if> -->
       <dynamics damping="0.0" friction="0.0"/>
     </joint>
@@ -176,15 +176,15 @@
       </sensor>
     </gazebo>
-    <joint name="${prefix}elbow_joint" type="revolute">
+    <joint name="${prefix}elbow_joint" type="continuous">
       <parent link="${prefix}upper_arm_link" />
       <child link = "${prefix}forearm_link" />
       <origin xyz="0.0 ${elbow_offset} ${upper_arm_length}" rpy="0.0 0.0 0.0" />
       <axis xyz="0 1 0" />
-      <xacro:unless value="${joint_limited}">
+      <!-- <xacro:unless value="${joint_limited}">
         <limit lower="${-0.75 * pi}" upper="${0.75 * pi}" effort="150.0" velocity="3.15"/>
       </xacro:unless>
       <xacro:if value="${joint_limited}">
         <limit lower="${-pi}" upper="${pi}" effort="150.0" velocity="3.15"/>
-      </xacro:if>
+      </xacro:if> -->
       <dynamics damping="0.0" friction="0.0"/>
     </joint>
@@ -221,15 +221,15 @@
       </sensor>
     </gazebo>
-    <joint name="${prefix}wrist_1_joint" type="revolute">
+    <joint name="${prefix}wrist_1_joint" type="continuous">
       <parent link="${prefix}forearm_link" />
       <child link = "${prefix}wrist_1_link" />
       <origin xyz="0.0 0.0 ${forearm_length}" rpy="0.0 ${pi / 2.0} 0.0" />
       <axis xyz="0 1 0" />
-      <xacro:unless value="${joint_limited}">
+      <!-- <xacro:unless value="${joint_limited}">
         <limit lower="${-2.0 * pi}" upper="${2.0 * pi}" effort="28.0" velocity="3.2"/>
       </xacro:unless>
       <xacro:if value="${joint_limited}">
         <limit lower="${-pi}" upper="${pi}" effort="28.0" velocity="3.2"/>
-      </xacro:if>
+      </xacro:if> -->
       <dynamics damping="0.0" friction="0.0"/>
     </joint>
@@ -266,15 +266,15 @@
       </sensor>
     </gazebo>
-    <joint name="${prefix}wrist_2_joint" type="revolute">
+    <joint name="${prefix}wrist_2_joint" type="continuous">
       <parent link="${prefix}wrist_1_link" />
       <child link = "${prefix}wrist_2_link" />
       <origin xyz="0.0 ${wrist_1_length} 0.0" rpy="0.0 0.0 0.0" />
       <axis xyz="0 0 1" />
-      <xacro:unless value="${joint_limited}">
+      <!-- <xacro:unless value="${joint_limited}">
         <limit lower="${-2.0 * pi}" upper="${2.0 * pi}" effort="28.0" velocity="3.2"/>
       </xacro:unless>
       <xacro:if value="${joint_limited}">
         <limit lower="${-pi}" upper="${pi}" effort="28.0" velocity="3.2"/>
-      </xacro:if>
+      </xacro:if> -->
       <dynamics damping="0.0" friction="0.0"/>
     </joint>
@@ -311,15 +311,15 @@
       </sensor>
     </gazebo>
-    <joint name="${prefix}wrist_3_joint" type="revolute">
+    <joint name="${prefix}wrist_3_joint" type="continuous">
       <parent link="${prefix}wrist_2_link" />
       <child link = "${prefix}wrist_3_link" />
       <origin xyz="0.0 0.0 ${wrist_2_length}" rpy="0.0 0.0 0.0" />
       <axis xyz="0 1 0" />
-      <xacro:unless value="${joint_limited}">
+      <!-- <xacro:unless value="${joint_limited}">
         <limit lower="${-2.0 * pi}" upper="${2.0 * pi}" effort="28.0" velocity="3.2"/>
       </xacro:unless>
       <xacro:if value="${joint_limited}">
         <limit lower="${-pi}" upper="${pi}" effort="28.0" velocity="3.2"/>
-      </xacro:if>
+      </xacro:if> -->
       <dynamics damping="0.0" friction="0.0"/>
     </joint>
